Commit message: urdf

File: src/vehicle_description/urdf/vehicle.xacro (robot description, xacro)
@@ -1,68 +1,90 @@
 <?xml version="1.0"?>
 <robot xmlns:xacro="http://www.ros.org/wiki/xacro" name="vehicle">
-  <!-- ================= BASE LINK ================= -->
+  <xacro:macro name="wheel" params="name x y">
+    <link name="${name}_wheel">
+      <visual>
+        <origin rpy="1.5708 0 0" xyz="0 0 0"/>
+        <geometry><cylinder length="0.1" radius="0.15"/></geometry>
+        <material name="black"><color rgba="0.1 0.1 0.1 1.0"/></material>
+      </visual>
+      <collision>
+        <origin rpy="1.5708 0 0" xyz="0 0 0"/>
+        <geometry><cylinder length="0.1" radius="0.15"/></geometry>
+      </collision>
+      <inertial>
+        <mass value="1.0"/>
+        <inertia ixx="0.01" iyy="0.01" izz="0.01" ixy="0" ixz="0" iyz="0"/>
+      </inertial>
+    </link>
+    <joint name="${name}_wheel_joint" type="continuous">
+      <parent link="base_link"/>
+      <child link="${name}_wheel"/>
+      <origin xyz="${x} ${y} -0.1"/>
+      <axis xyz="0 1 0"/>
+    </joint>
+  </xacro:macro>
   <link name="base_link">
     <visual>
-      <geometry>
-        <box size="1.0 0.6 0.2"/>
-      </geometry>
-      <material name="blue">
-        <color rgba="0.2 0.2 0.8 1.0"/>
-      </material>
+      <geometry><box size="1.0 0.6 0.2"/></geometry>
+      <material name="blue"><color rgba="0.2 0.2 0.8 1.0"/></material>
     </visual>
-    <collision>
-      <geometry>
-        <box size="1.0 0.6 0.2"/>
-      </geometry>
-    </collision>
+    <collision><geometry><box size="1.0 0.6 0.2"/></geometry></collision>
     <inertial>
-      <mass value="20.0"/>
-      <origin xyz="0 0 0"/>
-      <inertia ixx="1.0" iyy="1.0" izz="1.0"
-               ixy="0.0" ixz="0.0" iyz="0.0"/>
+      <mass value="15.0"/><origin xyz="0 0 0"/>
+      <inertia ixx="0.5" iyy="0.5" izz="0.5" ixy="0" ixz="0" iyz="0"/>
     </inertial>
   </link>
-  <!-- ================= LIDAR ================= -->
+  <xacro:wheel name="front_left"  x="0.35"  y="0.3"/>
+  <xacro:wheel name="front_right" x="0.35"  y="-0.3"/>
+  <xacro:wheel name="rear_left"   x="-0.35" y="0.3"/>
+  <xacro:wheel name="rear_right"  x="-0.35" y="-0.3"/>
   <link name="lidar_link">
-    <visual>
-      <geometry>
-        <cylinder radius="0.05" length="0.05"/>
-      </geometry>
-    </visual>
+    <visual><geometry><cylinder radius="0.05" length="0.05"/></geometry></visual>
+    <collision><geometry><cylinder radius="0.05" length="0.05"/></geometry></collision>
+    <inertial>
+      <mass value="0.1"/><origin xyz="0 0 0"/>
+      <inertia ixx="0.001" iyy="0.001" izz="0.001" ixy="0" ixz="0" iyz="0"/>
+    </inertial>
   </link>
   <joint name="lidar_joint" type="fixed">
-    <parent link="base_link"/>
-    <child link="lidar_link"/>
-    <origin xyz="0 0 0.2"/>
+    <parent link="base_link"/><child link="lidar_link"/><origin xyz="0 0 0.15"/>
   </joint>
   <gazebo reference="lidar_link">
-  <sensor type="ray" name="lidar">
-    <update_rate>10</update_rate>
-    <visualize>true</visualize>
-    <ray>
-      <scan>
-        <horizontal>
-          <samples>720</samples>
-          <min_angle>-3.14159</min_angle>
-          <max_angle>3.14159</max_angle>
-        </horizontal>
-      </scan>
-      <range>
-        <min>0.1</min>
-        <max>10.0</max>
-      </range>
-    </ray>
-    <!-- ✅ ROS2 Humble용 -->
-    <plugin
-      name="gazebo_ros_ray_sensor"
-      filename="libgazebo_ros_ray_sensor.so">
+    <sensor type="ray" name="lidar">
+      <update_rate>10</update_rate>
+      <visualize>true</visualize>
+      <ray>
+        <scan><horizontal><samples>360</samples><min_angle>-3.14</min_angle><max_angle>3.14</max_angle></horizontal></scan>
+        <range><min>0.1</min><max>12.0</max></range>
+      </ray>
+      <plugin name="gazebo_ros_laser" filename="libgazebo_ros_ray_sensor.so">
+        <ros>
+          <remapping>~/out:=scan</remapping>
+        </ros>
+        <output_type>sensor_msgs/LaserScan</output_type>
+        <frame_name>lidar_link</frame_name>
+      </plugin>
+    </sensor>
+  </gazebo>
+  <gazebo>
+    <plugin name="skid_steer_drive" filename="libgazebo_ros_diff_drive.so">
       <ros>
-        <namespace>/</namespace>
-        <remapping>~/out:=scan</remapping>
+        <remapping>odom:=odom</remapping>
       </ros>
-      <output_type>sensor_msgs/LaserScan</output_type>
-      <frame_name>lidar_link</frame_name>
+      <num_wheel_pairs>2</num_wheel_pairs>
+      <left_joint>front_left_wheel_joint</left_joint>
+      <right_joint>front_right_wheel_joint</right_joint>
+      <left_joint>rear_left_wheel_joint</left_joint>
+      <right_joint>rear_right_wheel_joint</right_joint>
+      <wheel_separation>0.6</wheel_separation>
+      <wheel_diameter>0.3</wheel_diameter>
+      <publish_odom>true</publish_odom>
+      <publish_odom_tf>true</publish_odom_tf>
+      <publish_wheel_tf>true</publish_wheel_tf>
+      <odometry_frame>odom</odometry_frame>
+      <robot_base_frame>base_link</robot_base_frame>
+      <max_wheel_torque>20</max_wheel_torque>
+      <max_wheel_acceleration>1.0</max_wheel_acceleration>
     </plugin>
-  </sensor>
-</gazebo>
+  </gazebo>
 </robot>

Commit message: ufdf2

File: src/vehicle_description/urdf/vehicle.xacro (robot description, xacro)
@@ -1,4 +1,32 @@
 <?xml version="1.0"?>
 <robot xmlns:xacro="http://www.ros.org/wiki/xacro" name="vehicle">
+  <xacro:macro name="wheel_inertia" params="m r h">
+    <inertial>
+      <mass value="${m}"/>
+      <inertia ixx="${(1/12)*m*(3*r*r + h*h)}" ixy="0" ixz="0"
+               iyy="${(1/12)*m*(3*r*r + h*h)}" iyz="0"
+               izz="${(1/2)*m*r*r}" />
+    </inertial>
+  </xacro:macro>
+  <link name="base_footprint"/>
+  <joint name="base_joint" type="fixed">
+    <parent link="base_footprint"/>
+    <child link="base_link"/>
+    <origin xyz="0 0 0.25" rpy="0 0 0"/>
+  </joint>
+  <link name="base_link">
+    <visual>
+      <geometry><box size="1.0 0.6 0.2"/></geometry>
+      <material name="blue"><color rgba="0.2 0.2 0.8 1.0"/></material>
+    </visual>
+    <collision><geometry><box size="1.0 0.6 0.2"/></geometry></collision>
+    <inertial>
+      <mass value="15.0"/>
+      <origin xyz="0 0 0"/>
+      <inertia ixx="${(1/12)*15.0*(0.6*0.6 + 0.2*0.2)}" ixy="0" ixz="0"
+               iyy="${(1/12)*15.0*(1.0*1.0 + 0.2*0.2)}" iyz="0"
+               izz="${(1/12)*15.0*(1.0*1.0 + 0.6*0.6)}" />
+    </inertial>
+  </link>
   <xacro:macro name="wheel" params="name x y">
     <link name="${name}_wheel">
@@ -12,8 +40,5 @@
         <geometry><cylinder length="0.1" radius="0.15"/></geometry>
       </collision>
-      <inertial>
-        <mass value="1.0"/>
-        <inertia ixx="0.01" iyy="0.01" izz="0.01" ixy="0" ixz="0" iyz="0"/>
-      </inertial>
+      <xacro:wheel_inertia m="1.0" r="0.15" h="0.1"/>
     </link>
     <joint name="${name}_wheel_joint" type="continuous">
@@ -24,15 +49,4 @@
     </joint>
   </xacro:macro>
-  <link name="base_link">
-    <visual>
-      <geometry><box size="1.0 0.6 0.2"/></geometry>
-      <material name="blue"><color rgba="0.2 0.2 0.8 1.0"/></material>
-    </visual>
-    <collision><geometry><box size="1.0 0.6 0.2"/></geometry></collision>
-    <inertial>
-      <mass value="15.0"/><origin xyz="0 0 0"/>
-      <inertia ixx="0.5" iyy="0.5" izz="0.5" ixy="0" ixz="0" iyz="0"/>
-    </inertial>
-  </link>
   <xacro:wheel name="front_left"  x="0.35"  y="0.3"/>
   <xacro:wheel name="front_right" x="0.35"  y="-0.3"/>
@@ -44,5 +58,5 @@
     <inertial>
       <mass value="0.1"/><origin xyz="0 0 0"/>
-      <inertia ixx="0.001" iyy="0.001" izz="0.001" ixy="0" ixz="0" iyz="0"/>
+      <inertia ixx="0.0001" iyy="0.0001" izz="0.0001" ixy="0" ixz="0" iyz="0"/>
     </inertial>
   </link>
@@ -50,4 +64,9 @@
     <parent link="base_link"/><child link="lidar_link"/><origin xyz="0 0 0.15"/>
   </joint>
+  <gazebo reference="base_link"><material>Gazebo/Blue</material></gazebo>
+  <gazebo reference="front_left_wheel"><material>Gazebo/Black</material></gazebo>
+  <gazebo reference="front_right_wheel"><material>Gazebo/Black</material></gazebo>
+  <gazebo reference="rear_left_wheel"><material>Gazebo/Black</material></gazebo>
+  <gazebo reference="rear_right_wheel"><material>Gazebo/Black</material></gazebo>
   <gazebo reference="lidar_link">
     <sensor type="ray" name="lidar">
@@ -56,10 +75,8 @@
       <ray>
         <scan><horizontal><samples>360</samples><min_angle>-3.14</min_angle><max_angle>3.14</max_angle></horizontal></scan>
-        <range><min>0.1</min><max>12.0</max></range>
+        <range><min>0.15</min><max>12.0</max></range>
       </ray>
       <plugin name="gazebo_ros_laser" filename="libgazebo_ros_ray_sensor.so">
-        <ros>
-          <remapping>~/out:=scan</remapping>
-        </ros>
+        <ros><remapping>~/out:=scan</remapping></ros>
         <output_type>sensor_msgs/LaserScan</output_type>
         <frame_name>lidar_link</frame_name>
@@ -68,22 +85,11 @@
   </gazebo>
   <gazebo>
-    <plugin name="skid_steer_drive" filename="libgazebo_ros_diff_drive.so">
-      <ros>
-        <remapping>odom:=odom</remapping>
-      </ros>
-      <num_wheel_pairs>2</num_wheel_pairs>
-      <left_joint>front_left_wheel_joint</left_joint>
-      <right_joint>front_right_wheel_joint</right_joint>
-      <left_joint>rear_left_wheel_joint</left_joint>
-      <right_joint>rear_right_wheel_joint</right_joint>
-      <wheel_separation>0.6</wheel_separation>
-      <wheel_diameter>0.3</wheel_diameter>
+    <plugin name="mecanum_drive" filename="libgazebo_ros_planar_move.so">
+      <ros><remapping>odom:=odom</remapping></ros>
+      <update_rate>50</update_rate>
       <publish_odom>true</publish_odom>
       <publish_odom_tf>true</publish_odom_tf>
-      <publish_wheel_tf>true</publish_wheel_tf>
       <odometry_frame>odom</odometry_frame>
-      <robot_base_frame>base_link</robot_base_frame>
-      <max_wheel_torque>20</max_wheel_torque>
-      <max_wheel_acceleration>1.0</max_wheel_acceleration>
+      <robot_base_frame>base_footprint</robot_base_frame> <publish_wheel_tf>true</publish_wheel_tf>
     </plugin>
   </gazebo>

Commit message: urdf3

File: src/vehicle_description/urdf/vehicle.xacro (robot description, xacro)
@@ -13,5 +13,5 @@
     <parent link="base_footprint"/>
     <child link="base_link"/>
-    <origin xyz="0 0 0.25" rpy="0 0 0"/>
+    <origin xyz="0 0 0.151" rpy="0 0 0"/>
   </joint>
   <link name="base_link">
@@ -45,7 +45,15 @@
       <parent link="base_link"/>
       <child link="${name}_wheel"/>
-      <origin xyz="${x} ${y} -0.1"/>
+      <origin xyz="${x} ${y} -0.151"/>
       <axis xyz="0 1 0"/>
     </joint>
+    <gazebo reference="${name}_wheel">
+      <material>Gazebo/Black</material>
+      <mu1>1.0</mu1>
+      <mu2>1.0</mu2>
+      <kp>1000000.0</kp>
+      <kd>100.0</kd>
+      <minDepth>0.001</minDepth>
+    </gazebo>
   </xacro:macro>
   <xacro:wheel name="front_left"  x="0.35"  y="0.3"/>
@@ -62,11 +70,7 @@
   </link>
   <joint name="lidar_joint" type="fixed">
-    <parent link="base_link"/><child link="lidar_link"/><origin xyz="0 0 0.15"/>
+    <parent link="base_link"/><child link="lidar_link"/><origin xyz="0 0 0.125"/>
   </joint>
   <gazebo reference="base_link"><material>Gazebo/Blue</material></gazebo>
-  <gazebo reference="front_left_wheel"><material>Gazebo/Black</material></gazebo>
-  <gazebo reference="front_right_wheel"><material>Gazebo/Black</material></gazebo>
-  <gazebo reference="rear_left_wheel"><material>Gazebo/Black</material></gazebo>
-  <gazebo reference="rear_right_wheel"><material>Gazebo/Black</material></gazebo>
   <gazebo reference="lidar_link">
     <sensor type="ray" name="lidar">
@@ -74,5 +78,5 @@
       <visualize>true</visualize>
       <ray>
-        <scan><horizontal><samples>360</samples><min_angle>-3.14</min_angle><max_angle>3.14</max_angle></horizontal></scan>
+        <scan><horizontal><samples>360</samples><min_angle>-3.14159</min_angle><max_angle>3.14159</max_angle></horizontal></scan>
         <range><min>0.15</min><max>12.0</max></range>
       </ray>
@@ -85,11 +89,22 @@
   </gazebo>
   <gazebo>
+    <plugin name="vehicle_joint_state" filename="libgazebo_ros_joint_state_publisher.so">
+      <ros><remapping>~/out:=joint_states</remapping></ros>
+      <update_rate>30</update_rate>
+      <joint_name>front_left_wheel_joint</joint_name>
+      <joint_name>front_right_wheel_joint</joint_name>
+      <joint_name>rear_left_wheel_joint</joint_name>
+      <joint_name>rear_right_wheel_joint</joint_name>
+    </plugin>
+  </gazebo>
+  <gazebo>
     <plugin name="mecanum_drive" filename="libgazebo_ros_planar_move.so">
       <ros><remapping>odom:=odom</remapping></ros>
-      <update_rate>50</update_rate>
+      <update_rate>100</update_rate>
       <publish_odom>true</publish_odom>
       <publish_odom_tf>true</publish_odom_tf>
       <odometry_frame>odom</odometry_frame>
-      <robot_base_frame>base_footprint</robot_base_frame> <publish_wheel_tf>true</publish_wheel_tf>
+      <robot_base_frame>base_footprint</robot_base_frame>
+      <publish_wheel_tf>false</publish_wheel_tf>
     </plugin>
   </gazebo>
